File: Zener and Led tester circuit.kicad_sch (KiCad schematic)
At the start: 15 parts, among them J1 Load, J2 Power supply, Q1 IRF840, U1 NE555P

Commit message: Zener and Led Tester Circuit is renewed
Other:
- company: (none) -> by Muxtar_Safarov
- title: (none) -> Zener and Led Tester Circuit 
Changed lines of the file:
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@@
 (kicad_sch (version 20230121) (generator eeschema)
   (paper "A4")
+  (title_block
+    (title "Zener and Led Tester Circuit ")
+    (date "21.12.2022")
+    (rev "1.0")
+    (company "by Muxtar_Safarov")
+  )
   (junction (at 138.43 44.45) (diameter 0) (color 0 0 0 0)
   )
